File: design_files/AST1031.brd (EAGLE design)
At the start: 9 x 16 mm, 12 parts, among them J1 SM05B, J4 SM02B-SRSS-TB(LF)(SN), U1 NCP2820

Commit message: updated documentation
Parts:
- C1: value 0.1uF -> 4.7uF; device tinycircuits:C0402 -> tinycircuits:C0603
- C2: value 10uF -> 0.1uF; device tinycircuits:C0603 -> tinycircuits:C0402
- J1: device tinycircuits:JST_SH_5X1 -> tinycircuits:JST_SH_5X1_EDGE
- moved C1 1.84 mm to (16.9, 18.4)
- moved C2 1.84 mm to (18.1, 17.1)
Other:
- board text added: "Wireling Audio Amp"
- board text removed: "Audio Board"
Changed lines of the file:
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@@
 <layer number="59" name="Invisible" color="7" fill="1" visible="no" active="no"/>
 <layer number="61" name="stand" color="7" fill="1" visible="no" active="no"/>
+<layer number="88" name="SimResults" color="9" fill="1" visible="yes" active="yes"/>
+<layer number="89" name="SimProbes" color="9" fill="1" visible="yes" active="yes"/>
 <layer number="90" name="Modules" color="5" fill="1" visible="yes" active="yes"/>
 <layer number="91" name="Nets" color="2" fill="1" visible="no" active="no"/>
@@
 <layer number="158" name="bResistor" color="7" fill="1" visible="yes" active="yes"/>
 <layer number="159" name="henwayCAP" color="13" fill="1" visible="yes" active="yes"/>
+<layer number="160" name="IDFDebug" color="7" fill="1" visible="yes" active="yes"/>
 <layer number="191" name="mNets" color="7" fill="1" visible="no" active="no"/>
 <layer number="192" name="mBusses" color="7" fill="1" visible="no" active="no"/>
@@
 <wire x1="0" y1="40.8" x2="0" y2="0" width="0.127" layer="48"/>
 <dimension x1="15.5" y1="26" x2="24.5" y2="26" x3="20" y3="27.454653125" layer="48"/>
-<text x="38.111025" y="4.365003125" size="0.889" layer="48">Audio Board</text>
+<text x="38.111025" y="4.365003125" size="0.889" layer="48">Wireling Audio Amp</text>
 <text x="34.986825" y="1.7714" size="0.889" layer="48">AS-PCB-AST1031</text>
 <text x="57.3810375" y="1.6952" size="0.889" layer="48">2</text>
@@
 <attribute name="NO_BOM" value="TRUE" x="34" y="0" size="1.778" layer="27" display="off"/>
 </element>
-<element name="C1" library="tinycircuits" package="C0402" value="0.1uF" x="18.15" y="17.05" rot="R90">
+<element name="C2" library="tinycircuits" package="C0402" value="0.1uF" x="18.15" y="17.05" rot="R90">
 <attribute name="PARTNO" value="AS-ITM-00008" x="18.15" y="17.05" size="1.778" layer="27" rot="R90" display="off"/>
 <attribute name="VALUE" value="0.1uF" x="18.15" y="17.05" size="1.778" layer="27" rot="R90" display="off"/>
 </element>
-<element name="C2" library="tinycircuits" package="C0603" value="10uF" x="16.9" y="18.4" rot="R90">
-<attribute name="PARTNO" value="AS-ITM-00002" x="16.9" y="18.4" size="1.778" layer="27" rot="R90" display="off"/>
-<attribute name="VALUE" value="10uF" x="16.9" y="18.4" size="1.778" layer="27" rot="R90" display="off"/>
+<element name="C1" library="tinycircuits" package="C0603" value="4.7uF" x="16.9" y="18.4" rot="R90">
+<attribute name="PARTNO" value="AS-ITM-00088" x="16.9" y="18.4" size="1.778" layer="27" rot="R90" display="off"/>
+<attribute name="VALUE" value="4.7uF" x="16.9" y="18.4" size="1.778" layer="27" rot="R90" display="off"/>
 </element>
-<element name="J1" library="tinycircuits" package="JST_SH_5X1" value="SM05B" x="20" y="12.125">
+<element name="J1" library="tinycircuits" package="JST_SH_5X1_EDGE" value="SM05B" x="20" y="12.125">
 <attribute name="PARTNO" value="AS-ITM-00340" x="20" y="12.125" size="1.778" layer="27" display="off"/>
 <attribute name="VALUE" value="SM05B" x="20" y="12.125" size="1.778" layer="27" display="off"/>
@@
 <vertex x="15.5" y="10"/>
 </polygon>
-<contactref element="C1" pad="2"/>
 <contactref element="C2" pad="2"/>
+<contactref element="C1" pad="2"/>
 <contactref element="J1" pad="1"/>
 <via x="18.1" y="10.8" extent="1-16" drill="0.381"/>
@@
 </signal>
 <signal name="VCC">
-<contactref element="C1" pad="1"/>
 <contactref element="C2" pad="1"/>
+<contactref element="C1" pad="1"/>
 <contactref element="J1" pad="2"/>
 <contactref element="U1" pad="6"/>
@@
 </signal>
 </signals>
-<errors>
-</errors>
 </board>
 </drawing>
