File: design_files/AST1031.sch (EAGLE design)
At the start: 11 parts, among them J1 SM05B, J4 SM02B-SRSS-TB(LF)(SN), U1 NCP2820

Commit message: updated documentation
Parts:
- C1: value 0.1uF -> 4.7uF; device tinycircuits:AS-ITM-00008 -> tinycircuits:AS-ITM-00088; PARTNO (none) -> AS-ITM-00088; VALUE (none) -> 4.7uF
- C2: value 10uF -> 0.1uF; device tinycircuits:AS-ITM-00002 -> tinycircuits:AS-ITM-00008
- J1: device tinycircuits:AS-ITM-00340 -> tinycircuits:AS-ITM-00340EDGE
Other:
- note added: "Wireling Audio Amp"
- note removed: "Audio Board"
- moved on the sheet: C1, C2
